File: Hardware/eNode_Spark.brd (EAGLE design)
At the start: 30 x 65 mm, 65 parts, among them U1 USD-SOCKETSMD, U10 WM-N-BM-09, U2 BMP180, U3 HTU21DSMD, U6 MCP73831T-2ACI/OT, U7 TMP006, U8 OPA344, U9 ADMP401, X1 USB-MICROB

Commit message: SOme routes added
Parts:
- moved LDR 63.7 mm to (28.0, 25.9), turned to 90.8 degrees
- moved R12 63.0 mm to (28.1, 21.4), turned to 268.6 degrees
- moved SV1 61.6 mm to (28.2, 14.1), turned to 271.3 degrees
- moved R11 58.3 mm to (25.9, 21.4), turned to 270.9 degrees
- moved C10 56.3 mm to (18.4, 21.5), turned to 272.3 degrees
- moved C12 56.3 mm to (14.6, 21.5), turned to 90.4 degrees
- moved C11 55.1 mm to (16.7, 24.3)
- moved C8 52.5 mm to (16.3, 21.5), turned to 93.3 degrees
- moved L1 49.9 mm to (12.4, 30.8)
- moved C9 48.8 mm to (5.63, 26.7)
Routing:
- net GND: track 0.00 -> 60.1 mm
- net +3V3: track 0.00 -> 25.4 mm
- net VBAT: track 0.00 -> 11.6 mm
- net RX: track 0.00 -> 11.4 mm
- net TX: track 0.00 -> 9.50 mm
- net UVCC: track 0.00 -> 2.80 mm
- net LDR: track 0.00 -> 2.66 mm
